File: 2401-pcb/2401-pcb.kicad_pcb (KiCad board)
At the start: 2 copper layers, 140 x 50 mm, 100 parts, among them J1 Load Cell, J2 Conn_ARM_JTAG_SWD_10, J3 Conn_01x04_Male, Q1 SFH3710, Q2 SFH3710, SW1 SW_SPDT, U1 LIS3DH, U10 MCP6001U, U11 MCP6001U, U2 VL6180X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

Commit message: Changes for production at aisler
Parts:
- C11, C12: value 4.7µF -> 4.7uF
- H1, H2: value MountingHole_Pad -> DNI
- J2: value Conn_ARM_JTAG_SWD_10 -> JTAG/SWD
- LOGO1, LOGO2, LOGO3: value LOGO -> DNI
- LOGO4: value LOGO -> DNI; footprint Logo:GND -> Jitter_Logos:Symbol_Jitter-Icon_CopperAndSilkScreenTop
- MB1, MB2, MB3, MB4: value Mousebite -> DNI
- Q1: value SFH3710 -> SFH3710(-Z)
- TH1, TH2, TH3, TH4: value ToolingHole -> DNI; footprint Jitter_Footprints:Tooling_hole_4mm_4.04mm_paste -> Jitter_Footprints:Tooling_hole_4.1mm_aisler
- U1: value LIS3DH -> LIS3DHTR
- U9: footprint Package_SO:SOIC-8_3.9x4.9mm_P1.27mm -> Package_SO:SOIC-8_5.275x5.275mm_P1.27mm
- moved C15 1.00 mm to (147.1, 125.6)
Routing:
- net /FLASH_MISO: track 14.6 -> 11.1 mm
- net /~FLASH_CS: track 11.3 -> 8.26 mm
- net +2V8: track 367.6 -> 370.3 mm
- net /FLASH_SCLK: track 15.9 -> 17.7 mm
- net /FLASH_MOSI: track 12.2 -> 13.0 mm

Commit message: PCb changes
Parts:
- R1: value 10M -> 1M
